Commit message: Add the metric release.v4 scene, the joint-space real replay and the V2 real eval.
- Scene airy_table_scene14sep26_left_image_metric: the release.v4 scene rescaled
  by 1.0915 about the camera, so sim distances match the real table.
- real_replay: record a sim grasp as joint_trajectory.npz, view it, replay it on
  the real RC5 by joints, locate the object with the ZED and render paired videos.
  The Cartesian NPZ replay stays as is.
- eval_openvla_v2_real.py plus eval_real_v2.sh: closed-loop OpenVLA-V2 eval with
  separate scene and wrist images and 7D proprio.
- eval_openvla_real.py: scene home joints, hand presets matched to the real
  AeroHand, and the home TCP read back from the controller.
- Hand visual profiles in config_debug.yaml, carried through the runner and the
  NPZ replay; joint4 URDF limit widened to +-360 deg for the real robot range.
- Docs for release.v4 and the joint replay, with tests for the scene and the
  hand materials.

Co-Authored-By: Claude Opus 5 <noreply@anthropic.com>

File: sim2real/openreal2sim/simulation/maniskill/robot_assets/rc5_aero_hand/urdf_rc5_right_hand/Robot _with_right_hand.urdf (robot description, URDF)
Before this commit: robot rc5_aero_hand, 40 links, 39 joints
Joints:
- joint joint3: limit lower=-3.14 upper=3.14 effort=50 velocity=1.5 -> lower=-6.283185 upper=6.283185 effort=50 velocity=1.5

File: sim2real/openreal2sim/simulation/maniskill/robot_assets/rc5_aero_hand/urdf_rc5_right_hand/Robot _with_right_hand_black_visual.urdf (robot description, URDF)
Before this commit: robot rc5_aero_hand, 40 links, 39 joints
Joints:
- joint joint3: limit lower=-3.14 upper=3.14 effort=50 velocity=1.5 -> lower=-6.283185 upper=6.283185 effort=50 velocity=1.5

File: sim2real/openreal2sim/simulation/maniskill/robot_assets/rc5_aero_hand/urdf_rc5_right_hand/Robot _with_right_hand_colored_visual.urdf (robot description, URDF)
Before this commit: robot rc5_aero_hand, 40 links, 39 joints
Joints:
- joint joint3: limit lower=-3.14 upper=3.14 effort=50 velocity=1.5 -> lower=-6.283185 upper=6.283185 effort=50 velocity=1.5

File: sim2real/openreal2sim/simulation/maniskill/robot_assets/rc5_aero_hand/urdf_rc5_right_hand/Robot _with_right_hand_colored_visual_continuous.urdf (robot description, URDF)
Before this commit: robot rc5_aero_hand, 40 links, 39 joints
Joints:
- joint joint3: limit lower=-3.14 upper=3.14 effort=50 velocity=1.5 -> lower=-6.283185 upper=6.283185 effort=50 velocity=1.5
